File: attempt.brd (EAGLE design)
At the start: 338.8 x 148.6 mm, 127 parts, among them J1 F-2X18-DIL-100, Q1 BSS138, Q10 BSS138, Q11 BSS138, Q15 BSS138, Q16 BSS138, Q17 BSS138, Q18 BSS138, Q19 BSS138, Q2 BSS138, Q20 BSS138, Q21 BSS138, Q22 BSS138, Q23 BSS138, Q24 BSS138, Q25 BSS138, Q26 BSS138, Q27 BSS138, Q28 BSS138, Q29 BSS138, Q3 BSS138, Q30 BSS138, Q4 BSS138, Q5 BSS138, Q6 BSS138, Q7 BSS138, Q8 BSS138, Q9 BSS138, U1 Value, U2 Value, X1 JST-XH-06-PIN-ROUND-PAD, X3 87758-0416, X4 87758-0616

Commit message: Add files via upload
Parts:
- removed BATTERY: 5566-2, con-molex:5566-2
- removed D1: (no value), sym:SOD123
- removed Q26, Q27, Q28, Q29, Q3, Q30: BSS138, Common-Parts-Library-Eagle:BSS138_SOT95P240X120-3N
- removed R12, R57, R58, R59, R60, R61, R62, R63, R64, R65, R66: 10k, adafruit:R0805
- removed X3: 87758-0416, con-molex:87758-0416
- added C8: 10uF, adafruit:C0805
- added C9: 1uF, Common-Parts-Library-Eagle:CC0603KRX7R9BB104_CAPC1608X90
- added J2: CLM-107-02-L-D-A, CLM-107-02-L-D-A:CLM10702LDA
- added J3: 53375-0610, wire to board_molex:53375-0610
- added JP10, JP11, JP8, JP9: (no value), pinhead:1X07
- added JP12: (no value), pinhead:1X02
- added S2, S3: E101SYZQE, SamacSys_Parts:E105MD9V3GE
- added U$1: XT60, XT60:XT60
- added U$3: IMU, IMU:PLCC28S
- added X2: 5566-4, con-molex:5566-4
- added Z1: MMSZ5256B-13-F, zener_diode:SOD3716X145N
- F2: value (none) -> MF-MSMF050-2; device fuse:GSH15 -> Common-Parts-Library-Eagle:MF-MSMF050-2_FUSM4632X85
- F3: value (none) -> MF-MSMF075-2; device fuse:GSH15 -> Common-Parts-Library-Eagle:FUSM4632X85
- R1: value 5k -> 56k
- R11: value 10k -> 5k
- RTC: value F-1X05-SIP-100-40 -> F-1X04-SIP-100-40; device con-headers-jp:SIP-100-05-40 -> con-headers-jp:SIP-100-04-40
- S1: value EG1213 -> E101SYZQE; device adafruit:EG1213 -> SamacSys_Parts:E105MD9V3GE
- X1: value JST-XH-06-PIN-ROUND-PAD -> 332-14; device Rembrandt Electronics - JST XH Connectors v1-0:JST-XH-06-PACKAGE-ROUND-PAD -> con-garry:332-14
- X4: value 87758-0616 -> (none); device con-molex:87758-0616 -> con-molex-micro-fit-3_0:43045-0600
- moved Q16 319.9 mm to (-246.3, -137.6)
- moved Q15 312.4 mm to (-238.7, -137.7), turned to 0 degrees
- moved Q17 307.4 mm to (-231.1, -138.0), turned to 0 degrees
- moved R6 214.4 mm to (-211.6, -77.1), turned to 180 degrees
- moved X1 205.0 mm to (-137.0, -112.5), turned to 0 degrees
- moved Q2 196.6 mm to (-134.4, -60.6), turned to 180 degrees
- moved C7 195.3 mm to (-175.1, -68.7), turned to 180 degrees
- moved C6 187.7 mm to (-175.4, -75.8), turned to 180 degrees
- moved HALL_3 187.7 mm to (-135.6, -52.5)
- moved Q22 186.2 mm to (-160.1, -59.8), turned to 180 degrees
- moved C5 185.1 mm to (-182.7, -76.3), turned to 180 degrees
- moved Q8 183.2 mm to (-151.4, -59.4), turned to 180 degrees
- moved IR_3 179.6 mm to (-149.1, -52.8)
- moved Q20 178.0 mm to (-146.9, -159.2), turned to 0 degrees
- moved ULTRA_4 176.7 mm to (-145.7, -166.8)
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Connections:
- removed net N$2: F2.1
- new net IN_JET: C2.1, S3.2, U1.1
- new net IN_SER: C4.1, R6.2, S2.2, U2.1
- new net N$28: JP8.4, U$3.22
- new net N$29: JP8.5, U$3.21
- new net N$31: JP8.6, U$3.20
- new net N$33: JP8.7, U$3.19
- new net N$35: JP9.2, U$3.17
- new net N$36: JP9.3, U$3.16
- new net N$37: JP9.4, U$3.15
- new net N$39: JP9.6, U$3.13
- new net N$40: JP9.7, U$3.12
- new net N$41: JP10.7, U$3.5
- new net N$43: JP10.5, U$3.7
- new net N$44: JP10.4, U$3.8
- new net N$45: JP10.3, U$3.9
- new net N$46: JP10.2, U$3.10
- new net N$47: JP10.1, U$3.11
- new net N$48: JP11.1, U$3.4
- new net N$49: JP11.2, U$3.3
- new net N$50: JP11.3, U$3.2
- new net N$51: JP11.4, U$3.1
- new net N$52: JP11.5, U$3.28
- new net N$53: JP11.6, U$3.27
- new net N$54: JP11.7, U$3.26
- new net N$55: HALL_3.3, Q8.3, R22.1
- new net N$56: HALL_4.3, Q9.3, R24.1
- new net N$58: F3.2, S3.1
- new net N$59: J2.1, X1.13
- new net N$60: J2.2, X1.14
- new net N$61: J2.3, X1.2
- new net N$62: J2.4, X1.4
- new net N$63: J2.5, X1.6
- new net N$64: J2.8, X1.1
- new net N$65: J2.6, X1.3
- new net TEMP_A6: JP12.2, JP3.7, R11.1
- net 3.3V: now also C8.1, C9.2, J2.11, X1.10, X1.11, X1.12; no longer Q26.1, Q27.1, Q28.1, Q29.1, Q3.1, Q30.1, R57.2, R59.2, R61.2, R63.2, R65.2
- net 5V: now also J3.2, RTC.3; no longer R12.2, R58.2, R60.2, R62.2, R64.2, R66.2, RTC.4, X1.2
- net 7.4V: now also J3.1; no longer X1.1
- net DATA_CONTROL_D7: now also J3.4; no longer X1.4
- net DIR_MOTOR_D2: no longer Q29.2, R63.1
- net EN_D3: no longer Q28.2, R61.1
- net GND: now also C8.2, C9.1, J2.13, J3.3, JP12.1, RTC.4, U$1.-, X1.7, X1.8, X1.9, X4.P$4, Z1.2; no longer BATTERY.2, D1.A, JP3.5, JP3.6, RTC.5, X1.3, X4.4
- net H1: now also X4.P$1; no longer X4.1
- net H2: now also X4.P$2; no longer X4.2
- net H3: now also X4.P$3; no longer X4.3
- net H_D34: no longer HALL_3.3, Q8.3, R22.1
- net H_D36: no longer HALL_4.3, Q9.3, R24.1
- net IN_1_D5: no longer Q26.2, R57.1
- net IN_2_D4: no longer Q27.2, R59.1
- net N$1: now also JP8.1, U$3.25; no longer JP3.8, Q30.2, R65.1
- net N$13: now also JP8.2, U$3.24; no longer Q29.3, R64.1
- net N$14: now also JP8.3, U$3.23; no longer Q3.3, R12.1
- net N$34: now also JP9.1, U$3.18; no longer Q26.3, R58.1
- net N$38: now also JP9.5, U$3.14; no longer Q27.3, R60.1
- net N$4: now also F2.2, S2.1; no longer F3.1
- net N$42: now also JP10.6, U$3.6; no longer Q28.3, R62.1
- net N$5: now also S1.2; no longer S1.3
- net READY_D6: no longer Q3.2, R11.1
- net RX3: now also J3.6; no longer X1.6
- net SCL_1: now also RTC.1; no longer RTC.2
- net SDA_1: now also RTC.2; no longer RTC.3
- net SET_A7: now also JP3.8; no longer Q30.3, R66.1
- net TX3: now also J3.5; no longer X1.5
- net VCC_HALL: now also X4.P$5; no longer X4.5
- net V_BATTERY: now also F2.1, F3.1, S1.1, U$1.+; no longer BATTERY.1, C2.1, C4.1, F2.2, F3.2, R6.2, S1.2, U1.1, U2.1
- net V_MOTOR: now also Z1.1; no longer D1.C
- net W1: now also X2.1; no longer X3.1
- net W2: now also X2.2; no longer X3.2
- net W3: now also X2.3; no longer X3.3
Other:
- board size 338.8 x 148.6 mm -> 175.6 x 121.4 mm
