File: attempt.brd (EAGLE design)
At the start: 338.8 x 148.6 mm, 127 parts, among them J1 F-2X18-DIL-100, Q1 BSS138, Q10 BSS138, Q11 BSS138, Q15 BSS138, Q16 BSS138, Q17 BSS138, Q18 BSS138, Q19 BSS138, Q2 BSS138, Q20 BSS138, Q21 BSS138, Q22 BSS138, Q23 BSS138, Q24 BSS138, Q25 BSS138, Q26 BSS138, Q27 BSS138, Q28 BSS138, Q29 BSS138, Q3 BSS138, Q30 BSS138, Q4 BSS138, Q5 BSS138, Q6 BSS138, Q7 BSS138, Q8 BSS138, Q9 BSS138, U1 Value, U2 Value, X1 JST-XH-06-PIN-ROUND-PAD, X3 87758-0416, X4 87758-0616

Commit message: Add files via upload
Parts:
- removed BATTERY: 5566-2, con-molex:5566-2
- removed D1: (no value), sym:SOD123
- removed F1: (no value), fuse:GSH15
- removed JP1: (no value), adafruit:2X09-BIG
- removed JP2, JP3, JP4, JP5, JP6, JP7: (no value), adafruit:1X08-BIG
- removed Q10, Q11, Q26, Q27, Q28, Q29, Q30: BSS138, Common-Parts-Library-Eagle:BSS138_SOT95P240X120-3N
- removed R25, R26, R27, R28, R57, R58, R59, R60, R61, R62, R63, R64, R65, R66: 10k, adafruit:R0805
- removed U$2: PINHD-1X10, adafruit:1X10-BIG
- removed X3: 87758-0416, con-molex:87758-0416
- added F4: SMF_OMNIBLOK_154.062, littlefuse_Nano2SMF_2:NANO2_SMF_FUSEBLOCK
- added J10, J2, J4, J5, J6, J7: F-1X08-SIP-100-32, con-headers-jp:SIP-100-08-32
- added J11: F-1X02-SIP-100-32, con-headers-jp:SIP-100-02-32
- added J3: 53375-0610, wire to board_molex:53375-0610
- added J8: F-1X10-SIP-100-32, con-headers-jp:SIP-100-10-32
- added J9: F-2X09-DIL-100, con-headers-jp:DIL-100-2X09
- added JP12: (no value), pinhead:1X02
- added R29: 1M, adafruit:R0805
- added S2, S3: E101SYZQE, SamacSys_Parts:E105MD9V3GE
- added U$1: XT60, XT60:XT60
- added X2: 5566-4, con-molex:5566-4
- added Z1: MMSZ5256B-13-F, zener_diode:SOD3716X145N
- F2: value (none) -> MF-MSMF050-2; device fuse:GSH15 -> Common-Parts-Library-Eagle:MF-MSMF050-2_FUSM4632X85
- F3: value (none) -> MF-MSMF075-2; device fuse:GSH15 -> Common-Parts-Library-Eagle:FUSM4632X85
- HALL_1, HALL_2, HALL_3, HALL_4: value F-1X04-SIP-100-40 -> F-1X03-SIP-100-32; device con-headers-jp:SIP-100-04-40 -> con-headers-jp:SIP-100-03-32
- IR_1, IR_2, IR_3, IR_4: value F-1X03-SIP-100-40 -> F-1X03-SIP-100-32; device con-headers-jp:SIP-100-03-40 -> con-headers-jp:SIP-100-03-32
- R1: value 5k -> 56k
- R10, R12, R13, R14, R15, R16, R17, R18, R19, R20, R21, R22, R23, R24, R35, R36, R37, R38, R39, R40, R41, R42, R43, R44, R45, R46, R47, R48, R49, R50, R51, R52, R53, R54, R55, R56, R7, R8, R9: value 10k -> 1M
- R11: value 10k -> 5k
- RTC: value F-1X05-SIP-100-40 -> F-1X04-SIP-100-32; device con-headers-jp:SIP-100-05-40 -> con-headers-jp:SIP-100-04-32
- S1: value EG1213 -> E101SYZQE; device adafruit:EG1213 -> SamacSys_Parts:E105MD9V3GE
- ULTRA_1, ULTRA_2, ULTRA_3, ULTRA_4: value F-1X04-SIP-100-40 -> F-1X04-SIP-100-32; device con-headers-jp:SIP-100-04-40 -> con-headers-jp:SIP-100-04-32
- X1: value JST-XH-06-PIN-ROUND-PAD -> TERMINAL-BLOCK-3.5MM-2-PIN-ROUND-PAD; device Rembrandt Electronics - JST XH Connectors v1-0:JST-XH-06-PACKAGE-ROUND-PAD -> Terminal Block 3-5mm v1-0:TERMINAL-BLOCK-2-PIN-3.5MM-ROUND-PAD
- X4: value 87758-0616 -> (none); device con-molex:87758-0616 -> con-molex-micro-fit-3_0:43045-0600
- moved HALL_1 488.9 mm to (159.5, 84.0)
- moved ULTRA_1 484.0 mm to (174.0, 76.0), turned to 270 degrees
- moved Q6 479.3 mm to (158.5, 78.0), turned to 0 degrees
- moved Q18 462.0 mm to (168.0, 78.0)
- moved IR_1 459.6 mm to (169.5, 63.5), turned to 270 degrees
- moved Q5 456.8 mm to (158.0, 61.5), turned to 270 degrees
- moved Q19 449.6 mm to (158.0, 70.1), turned to 270 degrees
- moved Q24 419.3 mm to (168.0, 10.5), turned to 270 degrees
- moved Q1 414.4 mm to (158.5, 29.0), turned to 270 degrees
- moved HALL_2 406.9 mm to (160.5, 5.00)
- moved IR_2 398.6 mm to (169.0, 27.5), turned to 90 degrees
- moved Q7 387.4 mm to (159.5, 11.0), turned to 180 degrees
- moved Q25 386.9 mm to (158.5, 19.6), turned to 270 degrees
- moved ULTRA_2 380.9 mm to (174.0, 11.0), turned to 90 degrees
- moved R17 346.1 mm to (142.4, 82.5), turned to 270 degrees
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Connections:
- removed net C_LIM: JP2.2, R1.2
- removed net DATA_CONTROL_D7: JP6.1, Q17.3, R40.1, X1.4
- removed net DIR_MOTOR_D2: JP2.4, JP6.6, Q29.2, R63.1
- removed net EN_D3: JP2.5, JP6.5, Q28.2, R61.1
- removed net IN_2_D4: JP2.6, JP6.4, Q27.2, R59.1
- removed net N$32: Q17.2, R39.1
- removed net N$34: Q26.3, R58.1
- removed net N$38: Q27.3, R60.1
- removed net N$42: Q28.3, R62.1
- removed net N$5 (its old number): F1.1, S1.3
- removed net READY_D6: JP2.8, JP6.2, Q3.2, R11.1
- removed net SCL_0: JP7.8
- removed net SCL_1: Q11.3, R28.1, RTC.2, U$2.1
- removed net SDA_0: JP7.7
- removed net SDA_1: Q10.3, R26.1, RTC.3, U$2.2
- new net DATA_CONTROL_D2: J6.6, Q17.2, R39.1
- new net DIR_MOTOR_D8: J10.4, J8.10
- new net EN_D7: J10.5, J6.1
- new net IN_2_D6: J10.6, J6.2
- new net IN_JET: C2.1, S3.2, U1.1
- new net IN_SER: C4.1, R6.2, S2.2, U2.1
- new net MOT_DATA_D3: J6.5, Q3.2, R29.1
- new net N$19: HALL_3.3, Q8.3, R22.1
- new net N$57: J9.18, Q3.3, R12.1
- new net N$58: F3.2, S3.1
- new net READY_D4: J10.8, J6.4
- new net TEMP_A6: J4.7, JP12.2, R11.1
- new net VCC: RTC.3
- net 3.3V: now also J2.4, R29.2; no longer JP4.4, Q10.1, Q11.1, Q26.1, Q27.1, Q28.1, Q29.1, Q30.1, R25.2, R27.2, R57.2, R59.2, R61.2, R63.2, R65.2
- net 5V: now also HALL_1.1, HALL_2.1, HALL_3.1, HALL_4.1, IR_1.1, IR_2.1, IR_3.1, IR_4.1, J2.5, J3.2, ULTRA_1.1, ULTRA_2.1, ULTRA_3.1, ULTRA_4.1; no longer HALL_1.4, HALL_2.4, HALL_3.4, HALL_4.4, IR_1.3, IR_2.3, IR_3.3, IR_4.3, JP4.5, R26.2, R28.2, R58.2, R60.2, R62.2, R64.2, R66.2, RTC.4, ULTRA_1.4, ULTRA_2.4, ULTRA_3.4, ULTRA_4.4, X1.2
- net 5V_JETSON: now also X1.1
- net 7.4V: now also J2.8, J3.1; no longer JP4.8, X1.1
- net GND: now also HALL_1.2, HALL_2.2, HALL_3.2, HALL_4.2, IR_1.2, IR_2.2, IR_3.2, IR_4.2, J10.3, J2.6, J2.7, J3.3, J9.14, J9.16, J9.9, JP12.1, RTC.4, U$1.-, ULTRA_1.4, ULTRA_2.4, ULTRA_3.4, ULTRA_4.4, X1.2, X4.P$4, Z1.2; no longer BATTERY.2, D1.A, HALL_1.1, HALL_2.1, HALL_3.1, HALL_4.1, IR_1.1, IR_2.1, IR_3.1, IR_4.1, JP1.9, JP2.3, JP3.5, JP3.6, JP4.6, JP4.7, RTC.5, ULTRA_1.1, ULTRA_2.1, ULTRA_3.1, ULTRA_4.1, X1.3, X4.4
- net H1: now also J9.13, X4.P$1; no longer JP1.13, X4.1
- net H2: now also J9.15, X4.P$2; no longer JP1.15, X4.2
- net H3: now also J9.17, X4.P$3; no longer JP1.17, X4.3
- net H_D34: no longer HALL_3.3, Q8.3, R22.1
- net H_D36: no longer HALL_4.3, Q9.3, R24.1
- net IN_1_D5: now also J10.7, J6.3; no longer JP2.7, JP6.3, Q26.2, R57.1
- net IR_D31: now also Q5.2, R15.1; no longer IR_1.2, Q5.3, R16.1
- net N$1: now also F4.2, S1.1; no longer JP3.8, Q30.2, R65.1
- net N$11: now also ULTRA_1.3; no longer ULTRA_1.2
- net N$12: now also IR_3.3; no longer IR_3.2
- net N$13: now also J11.1, RTC.1; no longer Q29.3, R64.1
- net N$14: now also J11.2, RTC.2; no longer Q3.3, R12.1
- net N$16: now also IR_4.3; no longer IR_4.2
- net N$17: now also J3.6, Q15.3, R36.1; no longer Q5.2, R15.1
- net N$18: now also ULTRA_4.2; no longer ULTRA_4.3
- net N$2: now also IR_1.3, Q5.3; no longer F2.1
- net N$20: now also ULTRA_4.3; no longer ULTRA_4.2
- net N$21: now also ULTRA_3.2; no longer ULTRA_3.3
- net N$22: now also ULTRA_3.3; no longer ULTRA_3.2
- net N$23: now also ULTRA_2.2; no longer ULTRA_2.3
- net N$24: now also HALL_4.3, Q9.3, R24.1; no longer Q10.2, R25.1
- net N$25: now also J10.2, R1.2; no longer Q11.2, R27.1
- net N$26: now also J3.5, Q16.3, R38.1; no longer Q15.2, R35.1
- net N$27: now also ULTRA_2.3; no longer ULTRA_2.2
- net N$30: now also J3.4, Q17.3, R40.1; no longer Q16.2, R37.1
- net N$4: now also F2.2, S2.1; no longer F3.1
- net N$7: now also IR_2.3; no longer IR_2.2
- net N$9: now also ULTRA_1.2; no longer ULTRA_1.3
- net RX3: now also J7.2, Q15.2, R35.1; no longer JP7.2, Q15.3, R36.1, X1.6
- net SET_A7: now also J10.1, J4.8; no longer JP2.1, Q30.3, R66.1
- net TX3: now also J7.1, Q16.2, R37.1; no longer JP7.1, Q16.3, R38.1, X1.5
- net VCC_HALL: now also J9.11, X4.P$5; no longer JP1.11, X4.5
- net V_BATTERY: now also F2.1, F3.1, F4.1, U$1.+; no longer BATTERY.1, C2.1, C4.1, F2.2, F3.2, R6.2, S1.2, U1.1, U2.1
- net V_MOTOR: now also J9.7, S1.2, Z1.1; no longer D1.C, F1.2, JP1.7
- net W1: now also J9.1, X2.1; no longer JP1.1, X3.1
- net W2: now also J9.3, X2.2; no longer JP1.3, X3.2
- net W3: now also J9.5, X2.3; no longer JP1.5, X3.3
Routing:
- removed copper zone on layer 16, net GND
Other:
- board size 338.8 x 148.6 mm -> 177 x 86 mm

Commit message: Add files via upload
Routing:
- net 5V: track 0.00 -> 529.9 mm, vias 0 -> 2
- net 3.3V: track 0.00 -> 461.4 mm, vias 0 -> 11
- net 7.4V: track 0.00 -> 165.9 mm, vias 0 -> 5
- net TEMP_A6: track 0.00 -> 143.0 mm, vias 0 -> 6
- net H_D30: track 0.00 -> 140.9 mm, vias 0 -> 9
- net TRIG_D22: track 0.00 -> 127.1 mm, vias 0 -> 6
- net IR_D37: track 0.00 -> 123.3 mm, vias 0 -> 6
- net TRIG_D28: track 0.00 -> 121.6 mm, vias 0 -> 6
- net SET_A7: track 0.00 -> 119.1 mm, vias 0 -> 3
- net H_D36: track 0.00 -> 113.8 mm, vias 0 -> 7
- net ECHO_D23: track 0.00 -> 111.0 mm, vias 0 -> 6
- net TRIG_D24: track 0.00 -> 94.6 mm, vias 0 -> 2
- net IR_D35: track 0.00 -> 88.2 mm, vias 0 -> 5
- net ECHO_D29: track 0.00 -> 87.6 mm, vias 0 -> 3
- net RX3: track 0.00 -> 84.9 mm, vias 0 -> 2
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- added copper zone on layer 1, net GND
- added copper zone on layer 16, net GND
Other:
- board size 177 x 86 mm -> 177 x 87 mm
