File: attempt.sch (EAGLE design)
At the start: 127 parts, among them J1 F-2X18-DIL-100, Q1 BSS138, Q10 BSS138, Q11 BSS138, Q15 BSS138, Q16 BSS138, Q17 BSS138, Q18 BSS138, Q19 BSS138, Q2 BSS138, Q20 BSS138, Q21 BSS138, Q22 BSS138, Q23 BSS138, Q24 BSS138, Q25 BSS138, Q26 BSS138, Q27 BSS138, Q28 BSS138, Q29 BSS138, Q3 BSS138, Q30 BSS138, Q4 BSS138, Q5 BSS138, Q6 BSS138, Q7 BSS138, Q8 BSS138, Q9 BSS138, U1 Value, U2 Value, X1 JST-XH-06-PIN-ROUND-PAD, X3 87758-0416, X4 87758-0616

Commit message: Add files via upload
Parts:
- removed BATTERY: 5566-2, con-molex:5566-2
- removed Q26, Q27, Q28, Q29, Q3, Q30: BSS138, Common-Parts-Library-Eagle:BSS138
- removed R12, R57, R58, R59, R60, R61, R62, R63, R64, R65, R66: 10k, adafruit:R-US_R0805
- removed X1: JST-XH-06-PIN-ROUND-PAD, Rembrandt Electronics - JST XH Connectors v1-0:JST-XH-06-PIN-ROUND-PAD
- added JP10, JP11, JP8, JP9: (no value), pinhead:PINHD-1X7
- added JP12: (no value), pinhead:PINHD-1X2
- added S2, S3: EG1213, adafruit:EG1213
- added SERVO: B6B-ZR, JST_1:B6B-ZR
- added U$1: XT60, XT60:XT60
- added U$3: IMU, IMU:IMU
- R11: value 10k -> 5k
- RTC: value F-1X05-SIP-100-40 -> F-1X04-SIP-100-40; device con-headers-jp:F-1X05-SIP-100-40 -> con-headers-jp:F-1X04-SIP-100-40
Connections:
- new net N$28: JP8.4, U$3.PIN_22
- new net N$29: JP8.5, U$3.PIN_21
- new net N$31: JP8.6, U$3.PIN_20
- new net N$33: JP8.7, U$3.PIN_19
- new net N$35: JP9.2, U$3.PIN_17
- new net N$36: JP9.3, U$3.PIN_16
- new net N$37: JP9.4, U$3.PIN_15
- new net N$39: JP9.6, U$3.PIN_13
- new net N$40: JP9.7, U$3.PIN_12
- new net N$41: JP10.7, U$3.PIN_5
- new net N$43: JP10.5, U$3.PIN_7
- new net N$44: JP10.4, U$3.PIN_8
- new net N$45: JP10.3, U$3.PIN_9
- new net N$46: JP10.2, U$3.PIN_10
- new net N$47: JP10.1, U$3.PIN_11
- new net N$48: JP11.1, U$3.PIN_4
- new net N$49: JP11.2, U$3.PIN_3
- new net N$50: JP11.3, U$3.PIN_2
- new net N$51: JP11.4, U$3.PIN_1
- new net N$52: JP11.5, U$3.PIN_28
- new net N$53: JP11.6, U$3.PIN_27
- new net N$54: JP11.7, U$3.PIN_26
- new net N$55: HALL_3.3, Q8.D, R22.1
- new net N$56: HALL_4.3, Q9.D, R24.1
- new net N$57: C4.1, R6.2, S21.S, U2.VIN
- new net N$58: C2.1, S31.S, U1.VIN
- new net TEMP_A6: JP12.2, JP3.7, R11.1
- net 3.3V: no longer Q26.G, Q27.G, Q28.G, Q29.G, Q3.G, Q30.G, R57.2, R59.2, R61.2, R63.2, R65.2
- net 5V: now also RTC.3, SERVO.2; no longer R12.2, R58.2, R60.2, R62.2, R64.2, R66.2, RTC.4, X1-2.S
- net 7.4V: now also SERVO.1; no longer X1-1.S
- net DATA_CONTROL_D7: now also SERVO.4; no longer X1-4.S
- net DIR_MOTOR_D2: no longer Q29.S, R63.1
- net EN_D3: no longer Q28.S, R61.1
- net GND: now also JP12.1, RTC.4, SERVO.3, U$1.GND; no longer BATTERY-2.S, JP3.5, JP3.6, RTC.5, X1-3.S
- net H_D34: no longer HALL_3.3, Q8.D, R22.1
- net H_D36: no longer HALL_4.3, Q9.D, R24.1
- net IN_1_D5: no longer Q26.S, R57.1
- net IN_2_D4: no longer Q27.S, R59.1
- net N$1: now also JP8.1, U$3.PIN_25; no longer JP3.8, Q30.S, R65.1
- net N$13: now also JP8.2, U$3.PIN_24; no longer Q29.D, R64.1
- net N$14: now also JP8.3, U$3.PIN_23; no longer Q3.D, R12.1
- net N$2: now also F2.2, S21.P; no longer F2.1
- net N$34: now also JP9.1, U$3.PIN_18; no longer Q26.D, R58.1
- net N$38: now also JP9.5, U$3.PIN_14; no longer Q27.D, R60.1
- net N$4: now also F3.2, S31.P; no longer F3.1
- net N$42: now also JP10.6, U$3.PIN_6; no longer Q28.D, R62.1
- net READY_D6: no longer Q3.S, R11.1
- net RX3: now also SERVO.6; no longer X1-6.S
- net SCL_1: now also RTC.1; no longer RTC.2
- net SDA_1: now also RTC.2; no longer RTC.3
- net SET_A7: now also JP3.8; no longer Q30.D, R66.1
- net TX3: now also SERVO.5; no longer X1-5.S
- net V_BATTERY: now also F2.1, F3.1, U$1.VCC; no longer BATTERY-1.S, C2.1, C4.1, F2.2, F3.2, R6.2, U1.VIN, U2.VIN
Other:
- moved on the sheet: F2, F3, R11
