File: attempt.sch (EAGLE design)
At the start: 127 parts, among them J1 F-2X18-DIL-100, Q1 BSS138, Q10 BSS138, Q11 BSS138, Q15 BSS138, Q16 BSS138, Q17 BSS138, Q18 BSS138, Q19 BSS138, Q2 BSS138, Q20 BSS138, Q21 BSS138, Q22 BSS138, Q23 BSS138, Q24 BSS138, Q25 BSS138, Q26 BSS138, Q27 BSS138, Q28 BSS138, Q29 BSS138, Q3 BSS138, Q30 BSS138, Q4 BSS138, Q5 BSS138, Q6 BSS138, Q7 BSS138, Q8 BSS138, Q9 BSS138, U1 Value, U2 Value, X1 JST-XH-06-PIN-ROUND-PAD, X3 87758-0416, X4 87758-0616

Commit message: Add files via upload
Parts:
- removed BATTERY: 5566-2, con-molex:5566-2
- removed D1: (no value), sym:ZENER
- removed Q26, Q27, Q28, Q29, Q3, Q30: BSS138, Common-Parts-Library-Eagle:BSS138
- removed R12, R57, R58, R59, R60, R61, R62, R63, R64, R65, R66: 10k, adafruit:R-US_R0805
- removed X1: JST-XH-06-PIN-ROUND-PAD, Rembrandt Electronics - JST XH Connectors v1-0:JST-XH-06-PIN-ROUND-PAD
- removed X3: 87758-0416, con-molex:87758-0416
- added C8: 10uF, adafruit:C-USC0805
- added C9: 1uF, Common-Parts-Library-Eagle:CC0603KRX7R9BB104
- added J2: CLM-107-02-L-D-A, CLM-107-02-L-D-A:CLM-107-02-L-D-A
- added J3: 53375-0610, wire to board_molex:53375-0610
- added J4: F-2X07-DIL-100, con-headers-jp:F-2X07-DIL-100
- added JP10, JP11, JP8, JP9: (no value), pinhead:PINHD-1X7
- added JP12: (no value), pinhead:PINHD-1X2
- added S2, S3: E101SYZQE, SamacSys_Parts:E101SYZQE
- added U$1: XT60, XT60:XT60
- added U$3: IMU, IMU:IMU
- added X2: 5566-4, con-molex:5566-4
- added Z1: MMSZ5256B-13-F, zener_diode:MMSZ5256B-13-F
- F2: value (none) -> MF-MSMF050-2; device fuse:GSH15 -> Common-Parts-Library-Eagle:MF-MSMF050-2
- F3: value (none) -> MF-MSMF075-2; device fuse:GSH15 -> Common-Parts-Library-Eagle:MF-MSMF075-2
- R1: value 5k -> 56k
- R11: value 10k -> 5k
- RTC: value F-1X05-SIP-100-40 -> F-1X04-SIP-100-40; device con-headers-jp:F-1X05-SIP-100-40 -> con-headers-jp:F-1X04-SIP-100-40
- S1: value EG1213 -> E101SYZQE; device adafruit:EG1213 -> SamacSys_Parts:E101SYZQE
- X4: value 87758-0616 -> (none); device con-molex:87758-0616 -> con-molex-micro-fit-3_0:HEADER_POS6_43045-0600
Connections:
- removed net N$2: F2.1
- new net IN_JET: C2.1, S3.2, U1.VIN
- new net IN_SER: C4.1, R6.2, S2.2, U2.VIN
- new net N$28: JP8.4, U$3.PIN_22
- new net N$29: JP8.5, U$3.PIN_21
- new net N$31: JP8.6, U$3.PIN_20
- new net N$33: JP8.7, U$3.PIN_19
- new net N$35: JP9.2, U$3.PIN_17
- new net N$36: JP9.3, U$3.PIN_16
- new net N$37: JP9.4, U$3.PIN_15
- new net N$39: JP9.6, U$3.PIN_13
- new net N$40: JP9.7, U$3.PIN_12
- new net N$41: JP10.7, U$3.PIN_5
- new net N$43: JP10.5, U$3.PIN_7
- new net N$44: JP10.4, U$3.PIN_8
- new net N$45: JP10.3, U$3.PIN_9
- new net N$46: JP10.2, U$3.PIN_10
- new net N$47: JP10.1, U$3.PIN_11
- new net N$48: JP11.1, U$3.PIN_4
- new net N$49: JP11.2, U$3.PIN_3
- new net N$50: JP11.3, U$3.PIN_2
- new net N$51: JP11.4, U$3.PIN_1
- new net N$52: JP11.5, U$3.PIN_28
- new net N$53: JP11.6, U$3.PIN_27
- new net N$54: JP11.7, U$3.PIN_26
- new net N$55: HALL_3.3, Q8.D, R22.1
- new net N$56: HALL_4.3, Q9.D, R24.1
- new net N$58: F3.2, S3.1
- new net N$59: J2.1, J4.13
- new net N$60: J2.2, J4.14
- new net N$61: J2.3, J4.2
- new net N$62: J2.4, J4.4
- new net N$63: J2.5, J4.6
- new net N$64: J2.8, J4.1
- new net N$65: J2.6, J4.3
- new net TEMP_A6: JP12.2, JP3.7, R11.1
- net 3.3V: now also C8.1, C9.2, J2.11, J4.10, J4.11, J4.12; no longer Q26.G, Q27.G, Q28.G, Q29.G, Q3.G, Q30.G, R57.2, R59.2, R61.2, R63.2, R65.2
- net 5V: now also J3.2, RTC.3; no longer R12.2, R58.2, R60.2, R62.2, R64.2, R66.2, RTC.4, X1-2.S
- net 7.4V: now also J3.1; no longer X1-1.S
- net DATA_CONTROL_D7: now also J3.4; no longer X1-4.S
- net DIR_MOTOR_D2: no longer Q29.S, R63.1
- net EN_D3: no longer Q28.S, R61.1
- net GND: now also C8.2, C9.1, J2.13, J3.3, J4.7, J4.8, J4.9, JP12.1, RTC.4, U$1.GND, X4.4, Z1.A; no longer BATTERY-2.S, D1.+, JP3.5, JP3.6, RTC.5, X1-3.S, X4-4.S
- net H1: now also X4.1; no longer X4-1.S
- net H2: now also X4.2; no longer X4-2.S
- net H3: now also X4.3; no longer X4-3.S
- net H_D34: no longer HALL_3.3, Q8.D, R22.1
- net H_D36: no longer HALL_4.3, Q9.D, R24.1
- net IN_1_D5: no longer Q26.S, R57.1
- net IN_2_D4: no longer Q27.S, R59.1
- net N$1: now also JP8.1, U$3.PIN_25; no longer JP3.8, Q30.S, R65.1
- net N$13: now also JP8.2, U$3.PIN_24; no longer Q29.D, R64.1
- net N$14: now also JP8.3, U$3.PIN_23; no longer Q3.D, R12.1
- net N$34: now also JP9.1, U$3.PIN_18; no longer Q26.D, R58.1
- net N$38: now also JP9.5, U$3.PIN_14; no longer Q27.D, R60.1
- net N$4: now also F2.2, S2.1; no longer F3.1
- net N$42: now also JP10.6, U$3.PIN_6; no longer Q28.D, R62.1
- net N$5: now also S1.2; no longer S11.S
- net READY_D6: no longer Q3.S, R11.1
- net RX3: now also J3.6; no longer X1-6.S
- net SCL_1: now also RTC.1; no longer RTC.2
- net SDA_1: now also RTC.2; no longer RTC.3
- net SET_A7: now also JP3.8; no longer Q30.D, R66.1
- net TX3: now also J3.5; no longer X1-5.S
- net VCC_HALL: now also X4.5; no longer X4-5.S
- net V_BATTERY: now also F2.1, F3.1, S1.1, U$1.VCC; no longer BATTERY-1.S, C2.1, C4.1, F2.2, F3.2, R6.2, S11.P, U1.VIN, U2.VIN
- net V_MOTOR: now also Z1.K; no longer D1.-
- net W1: now also X2-1.S; no longer X3-1.S
- net W2: now also X2-2.S; no longer X3-2.S
- net W3: now also X2-3.S; no longer X3-3.S
Other:
- moved on the sheet: R11
