File: attempt.sch (EAGLE design)
At the start: 127 parts, among them J1 F-2X18-DIL-100, Q1 BSS138, Q10 BSS138, Q11 BSS138, Q15 BSS138, Q16 BSS138, Q17 BSS138, Q18 BSS138, Q19 BSS138, Q2 BSS138, Q20 BSS138, Q21 BSS138, Q22 BSS138, Q23 BSS138, Q24 BSS138, Q25 BSS138, Q26 BSS138, Q27 BSS138, Q28 BSS138, Q29 BSS138, Q3 BSS138, Q30 BSS138, Q4 BSS138, Q5 BSS138, Q6 BSS138, Q7 BSS138, Q8 BSS138, Q9 BSS138, U1 Value, U2 Value, X1 JST-XH-06-PIN-ROUND-PAD, X3 87758-0416, X4 87758-0616

Commit message: Add files via upload
Parts:
- removed BATTERY: 5566-2, con-molex:5566-2
- removed D1: (no value), sym:ZENER
- removed F1: (no value), fuse:GSH15
- removed JP1: (no value), adafruit:PINHD-2X9-BIG
- removed JP2, JP3, JP4, JP5, JP6, JP7: (no value), adafruit:PINHD-1X8BIG
- removed Q26, Q27, Q28, Q29, Q30: BSS138, Common-Parts-Library-Eagle:BSS138
- removed R57, R58, R59, R60, R61, R62, R63, R64, R65, R66: 10k, adafruit:R-US_R0805
- removed U$2: PINHD-1X10, adafruit:PINHD-1X10
- removed X1: JST-XH-06-PIN-ROUND-PAD, Rembrandt Electronics - JST XH Connectors v1-0:JST-XH-06-PIN-ROUND-PAD
- removed X3: 87758-0416, con-molex:87758-0416
- added F4: SMF_OMNIBLOK_154.062, littlefuse_Nano2SMF_2:SMF_OMNIBLOK_154.062
- added J10, J2, J4, J5, J6, J7: F-1X08-SIP-100-32, con-headers-jp:F-1X08-SIP-100-32
- added J3: 53375-0610, wire to board_molex:53375-0610
- added J8: F-1X10-SIP-100-32, con-headers-jp:F-1X10-SIP-100-32
- added J9: F-2X09-DIL-100, con-headers-jp:F-2X09-DIL-100
- added JP12: (no value), pinhead:PINHD-1X2
- added R29: 10k, adafruit:R-US_R0805
- added S2, S3: E101SYZQE, SamacSys_Parts:E101SYZQE
- added U$1: XT60, XT60:XT60
- added X2: 5566-4, con-molex:5566-4
- added Z1: MMSZ5256B-13-F, zener_diode:MMSZ5256B-13-F
- F2: value (none) -> MF-MSMF050-2; device fuse:GSH15 -> Common-Parts-Library-Eagle:MF-MSMF050-2
- F3: value (none) -> MF-MSMF075-2; device fuse:GSH15 -> Common-Parts-Library-Eagle:MF-MSMF075-2
- HALL_1, HALL_2, HALL_3, HALL_4, ULTRA_1, ULTRA_2, ULTRA_3, ULTRA_4: value F-1X04-SIP-100-40 -> F-1X04-SIP-100-32; device con-headers-jp:F-1X04-SIP-100-40 -> con-headers-jp:F-1X04-SIP-100-32
- IR_1, IR_2, IR_3, IR_4: value F-1X03-SIP-100-40 -> F-1X04-SIP-100-32; device con-headers-jp:F-1X03-SIP-100-40 -> con-headers-jp:F-1X04-SIP-100-32
- R1: value 5k -> 56k
- R11: value 10k -> 5k
- RTC: value F-1X05-SIP-100-40 -> F-1X04-SIP-100-32; device con-headers-jp:F-1X05-SIP-100-40 -> con-headers-jp:F-1X04-SIP-100-32
- S1: value EG1213 -> E101SYZQE; device adafruit:EG1213 -> SamacSys_Parts:E101SYZQE
- X4: value 87758-0616 -> (none); device con-molex:87758-0616 -> con-molex-micro-fit-3_0:HEADER_POS6_43045-0600
Connections:
- net N$32 renamed DATA_CONTROL_D8
- removed net DATA_CONTROL_D7: JP6.1, Q17.D, R40.1, X1-4.S
- removed net N$1: JP3.8, Q30.S, R65.1
- removed net N$13: Q29.D, R64.1
- removed net N$14: Q3.D, R12.1
- removed net N$34: Q26.D, R58.1
- removed net N$38: Q27.D, R60.1
- removed net N$42: Q28.D, R62.1
- removed net SCL_0: JP7.8
- removed net SDA_0: JP7.7
- new net IN_JET: C2.1, S3.2, U1.VIN
- new net IN_SER: C4.1, R6.2, S2.2, U2.VIN
- new net MOT_DATA_D7: Q3.S, R29.1
- new net N$55: HALL_3.2, Q8.D, R22.1
- new net N$56: HALL_4.2, Q9.D, R24.1
- new net N$57: J9.18, Q3.D, R12.1
- new net N$58: F3.2, S3.1
- new net TEMP_A6: JP12.2, R11.1
- net 3.3V: now also R29.2; no longer JP4.4, Q26.G, Q27.G, Q28.G, Q29.G, Q30.G, R57.2, R59.2, R61.2, R63.2, R65.2
- net 5V: now also HALL_1.1, HALL_2.1, HALL_3.1, HALL_4.1, IR_1.1, IR_2.1, IR_3.1, IR_4.1, J3.2, RTC.2, ULTRA_1.1, ULTRA_2.1, ULTRA_3.1, ULTRA_4.1; no longer HALL_1.4, HALL_2.4, HALL_3.4, HALL_4.4, IR_1.3, IR_2.3, IR_3.3, IR_4.3, JP4.5, R58.2, R60.2, R62.2, R64.2, R66.2, RTC.4, ULTRA_1.4, ULTRA_2.4, ULTRA_3.4, ULTRA_4.4, X1-2.S
- net 7.4V: now also J3.1; no longer JP4.8, X1-1.S
- net C_LIM: now also J10.2; no longer JP2.2
- net DIR_MOTOR_D2: now also J10.4; no longer JP2.4, JP6.6, Q29.S, R63.1
- net EN_D3: now also J10.5; no longer JP2.5, JP6.5, Q28.S, R61.1
- net GND: now also HALL_1.4, HALL_2.4, HALL_3.4, HALL_4.4, IR_1.3, IR_2.3, IR_3.3, IR_4.3, J10.3, J3.3, J9.10, J9.14, J9.16, J9.9, JP12.1, RTC.1, U$1.GND, ULTRA_1.4, ULTRA_2.4, ULTRA_3.4, ULTRA_4.4, X4.4, Z1.A; no longer BATTERY-2.S, D1.+, HALL_1.1, HALL_2.1, HALL_3.1, HALL_4.1, IR_1.1, IR_2.1, IR_3.1, IR_4.1, JP1.9, JP2.3, JP3.5, JP3.6, JP4.6, JP4.7, RTC.5, ULTRA_1.1, ULTRA_2.1, ULTRA_3.1, ULTRA_4.1, X1-3.S, X4-4.S
- net H1: now also J9.13, X4.1; no longer JP1.13, X4-1.S
- net H2: now also J9.15, X4.2; no longer JP1.15, X4-2.S
- net H3: now also J9.17, X4.3; no longer JP1.17, X4-3.S
- net H_D34: no longer HALL_3.3, Q8.D, R22.1
- net H_D36: no longer HALL_4.3, Q9.D, R24.1
- net IN_1_D5: now also J10.7; no longer JP2.7, JP6.3, Q26.S, R57.1
- net IN_2_D4: now also J10.6; no longer JP2.6, JP6.4, Q27.S, R59.1
- net IR_D31: now also Q5.S, R15.1; no longer IR_1.2, Q5.D, R16.1
- net N$11: now also ULTRA_1.3; no longer ULTRA_1.2
- net N$15: now also HALL_2.2; no longer HALL_2.3
- net N$17: now also J3.6, Q15.D, R36.1; no longer Q5.S, R15.1
- net N$18: now also ULTRA_4.2; no longer ULTRA_4.3
- net N$19: now also HALL_1.2; no longer HALL_1.3
- net N$2: now also IR_1.2, Q5.D, R16.1; no longer F2.1
- net N$20: now also ULTRA_4.3; no longer ULTRA_4.2
- net N$21: now also ULTRA_3.2; no longer ULTRA_3.3
- net N$22: now also ULTRA_3.3; no longer ULTRA_3.2
- net N$23: now also ULTRA_2.2; no longer ULTRA_2.3
- net N$24: now also Q10.D, R26.1, RTC.3; no longer Q10.S, R25.1
- net N$25: now also Q11.D, R28.1, RTC.4; no longer Q11.S, R27.1
- net N$26: now also J3.5, Q16.D, R38.1; no longer Q15.S, R35.1
- net N$27: now also ULTRA_2.3; no longer ULTRA_2.2
- net N$30: now also J3.4, Q17.D, R40.1; no longer Q16.S, R37.1
- net N$4: now also F2.2, S2.1; no longer F3.1
- net N$5: now also F4.1, S1.2; no longer F1.1, S11.S
- net N$9: now also ULTRA_1.2; no longer ULTRA_1.3
- net READY_D6: now also J10.8; no longer JP2.8, JP6.2, Q3.S, R11.1
- net RX3: now also Q15.S, R35.1; no longer JP7.2, Q15.D, R36.1, X1-6.S
- net SCL_1: now also Q11.S, R27.1; no longer Q11.D, R28.1, RTC.2, U$2.1
- net SDA_1: now also Q10.S, R25.1; no longer Q10.D, R26.1, RTC.3, U$2.2
- net SET_A7: now also J10.1; no longer JP2.1, Q30.D, R66.1
- net TX3: now also Q16.S, R37.1; no longer JP7.1, Q16.D, R38.1, X1-5.S
- net VCC_HALL: now also J9.11, X4.5; no longer JP1.11, X4-5.S
- net V_BATTERY: now also F2.1, F3.1, S1.1, U$1.VCC; no longer BATTERY-1.S, C2.1, C4.1, F2.2, F3.2, R6.2, S11.P, U1.VIN, U2.VIN
- net V_MOTOR: now also F4.2, J9.7, J9.8, Z1.K; no longer D1.-, F1.2, JP1.7
- net W1: now also J9.1, J9.2, X2-1.S; no longer JP1.1, X3-1.S
- net W2: now also J9.3, J9.4, X2-2.S; no longer JP1.3, X3-2.S
- net W3: now also J9.5, J9.6, X2-3.S; no longer JP1.5, X3-3.S
Other:
- moved on the sheet: C1, C2, C3, HALL_1, HALL_2, HALL_3, HALL_4, R1, R11, R12, R2, R25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
